File: design.sch (KiCad schematic (older format))
At the start: 15 parts, among them J1 USB_C_Receptacle, J2 Conn_01x05, Q1 2N7002K, Q2 2N7002K, Q3 2N7002K, U1 ATtiny814-SS

Commit message: update
Connections:
- net Blue_PWM: now also U1.2 (PA4)
- net GND: now also C1.2, C2.2, J2.3 (Pin_3), U1.14 (GND)
- net Green_PWM: now also U1.3 (PA5)
- net Red_PWM: now also U1.6 (PB3)
- net WS2812b: now also U1.13 (PA3)
- net VCC: now reaches C1.1
- net VCC: now also C2.1, J2.2 (Pin_2), U1.1 (VCC)
- net UDPI: now reaches J2.1 (Pin_1)
- net UDPI: now also U1.10 (~RESET~/PA0)
- net TX: now reaches J2.4 (Pin_4)
- net TX: now also U1.11 (PA1)
- net RX: now reaches J2.5 (Pin_5)
- net RX: now also U1.12 (PA2)
Other:
- moved on the sheet: C1, C2
Changed lines of the file:
@@
 L Device:C_Small C1
 U 1 1 616F543B
-P 4650 2375
-F 0 "C1" H 4742 2421 50  0000 L CNN
-F 1 "C_Small" H 4742 2330 50  0000 L CNN
-F 2 "Capacitor_SMD:C_0805_2012Metric" H 4650 2375 50  0001 C CNN
-F 3 "~" H 4650 2375 50  0001 C CNN
-	1    4650 2375
+P 4725 2025
+F 0 "C1" H 4817 2071 50  0000 L CNN
+F 1 "C_Small" H 4817 1980 50  0000 L CNN
+F 2 "Capacitor_SMD:C_0805_2012Metric" H 4725 2025 50  0001 C CNN
+F 3 "~" H 4725 2025 50  0001 C CNN
+	1    4725 2025
 	1    0    0    -1
 $EndComp
@@
 L Device:C_Small C2
 U 1 1 616F58A4
-P 4325 2375
-F 0 "C2" H 4417 2421 50  0000 L CNN
-F 1 "C_Small" H 4417 2330 50  0000 L CNN
-F 2 "Capacitor_SMD:C_0805_2012Metric" H 4325 2375 50  0001 C CNN
-F 3 "~" H 4325 2375 50  0001 C CNN
-	1    4325 2375
+P 4400 2025
+F 0 "C2" H 4492 2071 50  0000 L CNN
+F 1 "C_Small" H 4492 1980 50  0000 L CNN
+F 2 "Capacitor_SMD:C_0805_2012Metric" H 4400 2025 50  0001 C CNN
+F 3 "~" H 4400 2025 50  0001 C CNN
+	1    4400 2025
 	1    0    0    -1
 $EndComp
@@
 Wire Wire Line
 	7700 4500 7700 4750
-Text GLabel 5675 3475 2    50   Input ~ 0
+Text GLabel 3975 3650 0    50   Input ~ 0
 Red_PWM
-Text GLabel 5675 3575 2    50   Input ~ 0
+Text GLabel 5175 3850 2    50   Input ~ 0
 Green_PWM
-Text GLabel 5675 3675 2    50   Input ~ 0
+Text GLabel 5175 3750 2    50   Input ~ 0
 Blue_PWM
 $Comp
@@
 Text GLabel 9475 4325 0    50   Input ~ 0
 WS2812b
-Text GLabel 5675 3875 2    50   Input ~ 0
+Text GLabel 5175 3650 2    50   Input ~ 0
 WS2812b
 $Comp
@@
 U 1 1 6179E4AD
 P 4575 3750
-F 0 "U1" H 4575 4631 50  0000 C CNN
-F 1 "ATtiny814-SS" H 4575 4540 50  0000 C CNN
+F 0 "U1" H 4800 4500 50  0000 C CNN
+F 1 "ATtiny814-SS" H 5000 4400 50  0000 C CNN
 F 2 "Package_SO:SOIC-14_3.9x8.7mm_P1.27mm" H 4575 3750 50  0001 C CIN
 F 3 "http://ww1.microchip.com/downloads/en/DeviceDoc/40001912A.pdf" H 4575 3750 50  0001 C CNN
@@
 	1    0    0    -1
 $EndComp
+Text GLabel 5175 3550 2    50   Input ~ 0
+RX
+Text GLabel 5175 3450 2    50   Input ~ 0
+TX
+Text GLabel 9300 2500 0    50   Input ~ 0
+RX
+Text GLabel 9300 2400 0    50   Input ~ 0
+TX
+Text GLabel 5175 3350 2    50   Input ~ 0
+UDPI
+Text GLabel 9300 2100 0    50   Input ~ 0
+UDPI
+$Comp
+L power:GND #PWR0104
+U 1 1 617577FD
+P 8775 2300
+F 0 "#PWR0104" H 8775 2050 50  0001 C CNN
+F 1 "GND" H 8780 2127 50  0000 C CNN
+F 2 "" H 8775 2300 50  0001 C CNN
+F 3 "" H 8775 2300 50  0001 C CNN
+	1    8775 2300
+	1    0    0    -1
+$EndComp
+Wire Wire Line
+	8775 2300 9300 2300
+$Comp
+L power:VCC #PWR0105
+U 1 1 61758559
+P 8775 2200
+F 0 "#PWR0105" H 8775 2050 50  0001 C CNN
+F 1 "VCC" H 8790 2373 50  0000 C CNN
+F 2 "" H 8775 2200 50  0001 C CNN
+F 3 "" H 8775 2200 50  0001 C CNN
+	1    8775 2200
+	1    0    0    -1
+$EndComp
+Wire Wire Line
+	8775 2200 9300 2200
+$Comp
+L power:VCC #PWR0106
+U 1 1 6175914C
+P 4575 3050
+F 0 "#PWR0106" H 4575 2900 50  0001 C CNN
+F 1 "VCC" H 4590 3223 50  0000 C CNN
+F 2 "" H 4575 3050 50  0001 C CNN
+F 3 "" H 4575 3050 50  0001 C CNN
+	1    4575 3050
+	1    0    0    -1
+$EndComp
+$Comp
+L power:VCC #PWR0107
+U 1 1 6175A657
+P 4575 1700
+F 0 "#PWR0107" H 4575 1550 50  0001 C CNN
+F 1 "VCC" H 4590 1873 50  0000 C CNN
+F 2 "" H 4575 1700 50  0001 C CNN
+F 3 "" H 4575 1700 50  0001 C CNN
+	1    4575 1700
+	1    0    0    -1
+$EndComp
+$Comp
+L power:GND #PWR0108
+U 1 1 6175AB45
+P 4575 4450
+F 0 "#PWR0108" H 4575 4200 50  0001 C CNN
+F 1 "GND" H 4580 4277 50  0000 C CNN
+F 2 "" H 4575 4450 50  0001 C CNN
+F 3 "" H 4575 4450 50  0001 C CNN
+	1    4575 4450
+	1    0    0    -1
+$EndComp
+$Comp
+L power:GND #PWR0109
+U 1 1 6175B11F
+P 4575 2250
+F 0 "#PWR0109" H 4575 2000 50  0001 C CNN
+F 1 "GND" H 4580 2077 50  0000 C CNN
+F 2 "" H 4575 2250 50  0001 C CNN
+F 3 "" H 4575 2250 50  0001 C CNN
+	1    4575 2250
+	1    0    0    -1
+$EndComp
+Wire Wire Line
+	4400 2125 4400 2250
+Wire Wire Line
+	4400 2250 4575 2250
+Wire Wire Line
+	4575 2250 4725 2250
+Wire Wire Line
+	4725 2250 4725 2125
+Connection ~ 4575 2250
+Wire Wire Line
+	4725 1925 4725 1700
+Wire Wire Line
+	4725 1700 4575 1700
+Wire Wire Line
+	4575 1700 4400 1700
+Wire Wire Line
+	4400 1700 4400 1925
+Connection ~ 4575 1700
 $EndSCHEMATC

Commit message: add components
usb resistor cc, power flags, mosfet gate resistor
Parts:
- added R? (x3): R_Small, Resistor_SMD:R_0805_2012Metric, symbol Device:R_Small
- added R? (x2): 5.1k, Resistor_SMD:R_0805_2012Metric, symbol Device:R_Small
Connections:
- net Blue_PWM: now also R?.1; no longer Q3.1 (G), R3.1
- net GND: now also J1.A1 (GND), J1.A12 (GND), J1.B1 (GND), J1.B12 (GND), J1.S1 (SHIELD), R?.2, R?.2
- net Green_PWM: now also R?.1; no longer Q2.1 (G), R2.1
- net Red_PWM: now also R?.1; no longer Q1.1 (G), R1.1
- net VCC: now also J1.A4 (VBUS), J1.A9 (VBUS), J1.B4 (VBUS), J1.B9 (VBUS)
- net at J1.A5 (CC1): now also R?.1
- net at J1.B5 (CC2): now also R?.1
- new net: Q1.1 (G), R1.1, R?.2
- new net: Q2.1 (G), R2.1, R?.2
- new net: Q3.1 (G), R3.1, R?.2
- no-connect marks 0 -> 14
Changed lines of the file:
@@
 	7125 2675 7675 2675
 Connection ~ 7675 2675
-Text GLabel 7000 2475 0    50   Input ~ 0
+Text GLabel 6675 2475 0    50   Input ~ 0
 Red_PWM
-Text GLabel 7025 3675 0    50   Input ~ 0
+Text GLabel 6700 3675 0    50   Input ~ 0
 Green_PWM
-Text GLabel 7000 4950 0    50   Input ~ 0
+Text GLabel 6675 4950 0    50   Input ~ 0
 Blue_PWM
 Wire Wire Line
@@
 	4400 1700 4400 1925
 Connection ~ 4575 1700
+$Comp
+L Device:R_Small R?
+U 1 1 61A6A719
+P 6900 2475
+F 0 "R?" H 6959 2521 50  0000 L CNN
+F 1 "R_Small" H 6959 2430 50  0000 L CNN
+F 2 "Resistor_SMD:R_0805_2012Metric" H 6900 2475 50  0001 C CNN
+F 3 "~" H 6900 2475 50  0001 C CNN
+	1    6900 2475
+	0    -1   -1   0
+$EndComp
+Wire Wire Line
+	6675 2475 6800 2475
+$Comp
+L Device:R_Small R?
+U 1 1 61A6CC22
+P 6925 3675
+F 0 "R?" H 6984 3721 50  0000 L CNN
+F 1 "R_Small" H 6984 3630 50  0000 L CNN
+F 2 "Resistor_SMD:R_0805_2012Metric" H 6925 3675 50  0001 C CNN
+F 3 "~" H 6925 3675 50  0001 C CNN
+	1    6925 3675
+	0    -1   -1   0
+$EndComp
+Wire Wire Line
+	6700 3675 6825 3675
+$Comp
+L Device:R_Small R?
+U 1 1 61A6D9D6
+P 6900 4950
+F 0 "R?" H 6959 4996 50  0000 L CNN
+F 1 "R_Small" H 6959 4905 50  0000 L CNN
+F 2 "Resistor_SMD:R_0805_2012Metric" H 6900 4950 50  0001 C CNN
+F 3 "~" H 6900 4950 50  0001 C CNN
+	1    6900 4950
+	0    -1   -1   0
+$EndComp
+Wire Wire Line
+	6675 4950 6800 4950
+NoConn ~ 2700 3075
+NoConn ~ 2700 3175
+NoConn ~ 2700 3275
+NoConn ~ 2700 3375
+NoConn ~ 2700 3575
+NoConn ~ 2700 3675
+NoConn ~ 2700 3875
+NoConn ~ 2700 3975
+NoConn ~ 2700 4175
+NoConn ~ 2700 4275
+NoConn ~ 2700 4475
+NoConn ~ 2700 4575
+NoConn ~ 2700 4775
+NoConn ~ 2700 4875
+$Comp
+L power:GND #PWR?
+U 1 1 61A7334E
+P 1925 5375
+F 0 "#PWR?" H 1925 5125 50  0001 C CNN
+F 1 "GND" H 1930 5202 50  0000 C CNN
+F 2 "" H 1925 5375 50  0001 C CNN
+F 3 "" H 1925 5375 50  0001 C CNN
+	1    1925 5375
+	1    0    0    -1
+$EndComp
+Wire Wire Line
+	1925 5375 1800 5375
+Wire Wire Line
+	1800 5375 1800 5175
+Wire Wire Line
+	1925 5375 2100 5375
+Wire Wire Line
+	2100 5375 2100 5175
+Connection ~ 1925 5375
+$Comp
+L power:VCC #PWR?
+U 1 1 61A74E6E
+P 2975 2575
+F 0 "#PWR?" H 2975 2425 50  0001 C CNN
+F 1 "VCC" H 2990 2748 50  0000 C CNN
+F 2 "" H 2975 2575 50  0001 C CNN
+F 3 "" H 2975 2575 50  0001 C CNN
+	1    2975 2575
+	1    0    0    -1
+$EndComp
+Wire Wire Line
+	2975 2575 2700 2575
+$Comp
+L Device:R_Small R?
+U 1 1 61A75EA7
+P 3175 2775
+F 0 "R?" H 3234 2821 50  0000 L CNN
+F 1 "5.1k" H 3234 2730 50  0000 L CNN
+F 2 "Resistor_SMD:R_0805_2012Metric" H 3175 2775 50  0001 C CNN
+F 3 "~" H 3175 2775 50  0001 C CNN
+	1    3175 2775
+	0    -1   -1   0
+$EndComp
+Wire Wire Line
+	3075 2775 2700 2775
+Wire Wire Line
+	2700 2875 3075 2875
+$Comp
+L Device:R_Small R?
+U 1 1 61A77F57
+P 3175 2875
+F 0 "R?" H 3000 2925 50  0000 L CNN
+F 1 "5.1k" H 2950 2825 50  0000 L CNN
+F 2 "Resistor_SMD:R_0805_2012Metric" H 3175 2875 50  0001 C CNN
+F 3 "~" H 3175 2875 50  0001 C CNN
+	1    3175 2875
+	0    -1   -1   0
+$EndComp
+$Comp
+L power:GND #PWR?
+U 1 1 61A78369
+P 3525 2825
+F 0 "#PWR?" H 3525 2575 50  0001 C CNN
+F 1 "GND" H 3530 2652 50  0000 C CNN
+F 2 "" H 3525 2825 50  0001 C CNN
+F 3 "" H 3525 2825 50  0001 C CNN
+	1    3525 2825
+	1    0    0    -1
+$EndComp
+Wire Wire Line
+	3275 2875 3375 2875
+Wire Wire Line
+	3375 2875 3375 2825
+Wire Wire Line
+	3375 2825 3525 2825
+Wire Wire Line
+	3375 2825 3375 2775
+Wire Wire Line
+	3375 2775 3275 2775
+Connection ~ 3375 2825
 $EndSCHEMATC

Commit message: Revert "add components"
This reverts commit 60fcf040a8541399063354e6f95bf0141af0d636.
Parts:
- removed R? (x3): R_Small, Resistor_SMD:R_0805_2012Metric, symbol Device:R_Small
- removed R? (x2): 5.1k, Resistor_SMD:R_0805_2012Metric, symbol Device:R_Small
Connections:
- net Blue_PWM: now also Q3.1 (G), R3.1
- net GND: no longer J1.A1 (GND), J1.A12 (GND), J1.B1 (GND), J1.B12 (GND), J1.S1 (SHIELD)
- net Green_PWM: now also Q2.1 (G), R2.1
- net Red_PWM: now also Q1.1 (G), R1.1
- net VCC: no longer J1.A4 (VBUS), J1.A9 (VBUS), J1.B4 (VBUS), J1.B9 (VBUS)
- new net: J1.A1 (GND), J1.A12 (GND), J1.B1 (GND), J1.B12 (GND)
- new net: J1.A4 (VBUS), J1.A9 (VBUS), J1.B4 (VBUS), J1.B9 (VBUS)
- no-connect marks 14 -> 0
Changed lines of the file:
@@
 	7125 2675 7675 2675
 Connection ~ 7675 2675
-Text GLabel 6675 2475 0    50   Input ~ 0
+Text GLabel 7000 2475 0    50   Input ~ 0
 Red_PWM
-Text GLabel 6700 3675 0    50   Input ~ 0
+Text GLabel 7025 3675 0    50   Input ~ 0
 Green_PWM
-Text GLabel 6675 4950 0    50   Input ~ 0
+Text GLabel 7000 4950 0    50   Input ~ 0
 Blue_PWM
 Wire Wire Line
@@
 	4400 1700 4400 1925
 Connection ~ 4575 1700
-$Comp
-L Device:R_Small R?
-U 1 1 61A6A719
-P 6900 2475
-F 0 "R?" H 6959 2521 50  0000 L CNN
-F 1 "R_Small" H 6959 2430 50  0000 L CNN
-F 2 "Resistor_SMD:R_0805_2012Metric" H 6900 2475 50  0001 C CNN
-F 3 "~" H 6900 2475 50  0001 C CNN
-	1    6900 2475
-	0    -1   -1   0
-$EndComp
-Wire Wire Line
-	6675 2475 6800 2475
-$Comp
-L Device:R_Small R?
-U 1 1 61A6CC22
-P 6925 3675
-F 0 "R?" H 6984 3721 50  0000 L CNN
-F 1 "R_Small" H 6984 3630 50  0000 L CNN
-F 2 "Resistor_SMD:R_0805_2012Metric" H 6925 3675 50  0001 C CNN
-F 3 "~" H 6925 3675 50  0001 C CNN
-	1    6925 3675
-	0    -1   -1   0
-$EndComp
-Wire Wire Line
-	6700 3675 6825 3675
-$Comp
-L Device:R_Small R?
-U 1 1 61A6D9D6
-P 6900 4950
-F 0 "R?" H 6959 4996 50  0000 L CNN
-F 1 "R_Small" H 6959 4905 50  0000 L CNN
-F 2 "Resistor_SMD:R_0805_2012Metric" H 6900 4950 50  0001 C CNN
-F 3 "~" H 6900 4950 50  0001 C CNN
-	1    6900 4950
-	0    -1   -1   0
-$EndComp
-Wire Wire Line
-	6675 4950 6800 4950
-NoConn ~ 2700 3075
-NoConn ~ 2700 3175
-NoConn ~ 2700 3275
-NoConn ~ 2700 3375
-NoConn ~ 2700 3575
-NoConn ~ 2700 3675
-NoConn ~ 2700 3875
-NoConn ~ 2700 3975
-NoConn ~ 2700 4175
-NoConn ~ 2700 4275
-NoConn ~ 2700 4475
-NoConn ~ 2700 4575
-NoConn ~ 2700 4775
-NoConn ~ 2700 4875
-$Comp
-L power:GND #PWR?
-U 1 1 61A7334E
-P 1925 5375
-F 0 "#PWR?" H 1925 5125 50  0001 C CNN
-F 1 "GND" H 1930 5202 50  0000 C CNN
-F 2 "" H 1925 5375 50  0001 C CNN
-F 3 "" H 1925 5375 50  0001 C CNN
-	1    1925 5375
-	1    0    0    -1
-$EndComp
-Wire Wire Line
-	1925 5375 1800 5375
-Wire Wire Line
-	1800 5375 1800 5175
-Wire Wire Line
-	1925 5375 2100 5375
-Wire Wire Line
-	2100 5375 2100 5175
-Connection ~ 1925 5375
-$Comp
-L power:VCC #PWR?
-U 1 1 61A74E6E
-P 2975 2575
-F 0 "#PWR?" H 2975 2425 50  0001 C CNN
-F 1 "VCC" H 2990 2748 50  0000 C CNN
-F 2 "" H 2975 2575 50  0001 C CNN
-F 3 "" H 2975 2575 50  0001 C CNN
-	1    2975 2575
-	1    0    0    -1
-$EndComp
-Wire Wire Line
-	2975 2575 2700 2575
-$Comp
-L Device:R_Small R?
-U 1 1 61A75EA7
-P 3175 2775
-F 0 "R?" H 3234 2821 50  0000 L CNN
-F 1 "5.1k" H 3234 2730 50  0000 L CNN
-F 2 "Resistor_SMD:R_0805_2012Metric" H 3175 2775 50  0001 C CNN
-F 3 "~" H 3175 2775 50  0001 C CNN
-	1    3175 2775
-	0    -1   -1   0
-$EndComp
-Wire Wire Line
-	3075 2775 2700 2775
-Wire Wire Line
-	2700 2875 3075 2875
-$Comp
-L Device:R_Small R?
-U 1 1 61A77F57
-P 3175 2875
-F 0 "R?" H 3000 2925 50  0000 L CNN
-F 1 "5.1k" H 2950 2825 50  0000 L CNN
-F 2 "Resistor_SMD:R_0805_2012Metric" H 3175 2875 50  0001 C CNN
-F 3 "~" H 3175 2875 50  0001 C CNN
-	1    3175 2875
-	0    -1   -1   0
-$EndComp
-$Comp
-L power:GND #PWR?
-U 1 1 61A78369
-P 3525 2825
-F 0 "#PWR?" H 3525 2575 50  0001 C CNN
-F 1 "GND" H 3530 2652 50  0000 C CNN
-F 2 "" H 3525 2825 50  0001 C CNN
-F 3 "" H 3525 2825 50  0001 C CNN
-	1    3525 2825
-	1    0    0    -1
-$EndComp
-Wire Wire Line
-	3275 2875 3375 2875
-Wire Wire Line
-	3375 2875 3375 2825
-Wire Wire Line
-	3375 2825 3525 2825
-Wire Wire Line
-	3375 2825 3375 2775
-Wire Wire Line
-	3375 2775 3275 2775
-Connection ~ 3375 2825
 $EndSCHEMATC
